File: Hardware/SparkFun LoRaSerial - 1W.sch (EAGLE design)
At the start: 56 parts, among them J1 QWIIC_RIGHT_ANGLE, J3 USB C, J4 JTAG, U2 ATSAMD21G-A, U3 AP2112K-3.3, U4 E19-915M30S, Y1 32.768kHz

Commit message: File rename
Parts:
- added S1: Reset, SparkFun-Switches:MOMENTARY-SWITCH-SPST-SMD-RIGHT-ANGLE
Connections:
- net BOARD_ID renamed A2/BOARD_ID
- net SPI_PICO renamed D11/SPI_PICO
- net SPI_POCI renamed D12/SPI_POCI
- net SPI_SCK renamed D13/SPI_SCK
- removed net A3: U2.PA04(AIN4/REFB/SER0:0/TC0:0)
- new net A3/TRAIN: S1.2, U2.PA04(AIN4/REFB/SER0:0/TC0:0)
- new net A4: U2.PA05(AIN5/SER0:1/TC0:1)
- new net A5: U2.PB02(AIN10/SER5:0)
- new net D30: U2.PB22(SER5:2+)
- new net D31: U2.PB23(SER5:3+)
- net GND: now also S1.1
- net RX_LED: no longer U2.PB03(AIN11/SER5:1)
- net TX_LED: no longer U2.PA27
Other:
- note added: "Add CTS RTS connections to GPIOs"
- note added: "Add PTH holes for GPIO"
- note added: "Add train button"
- note added: "Bootloader RX LED"
- note added: "Bootloader TX LED"
- note added: "Do we need to move the TX/RX LEDs from the USB so they work during external radio connection?"
- note removed: "PA12 is SPI MISO (on SPI header)."
- note removed: "PA13 is DGI GPIO0 (goes to EDBG)."
- note removed: "PA5 is A4"
- note removed: "PB10/11 are MOSI/SCK to SPI header."
- note removed: "PB2 is A5"
- note removed: "PB22/23 are TXD/RXD to the EDBG"
Changed lines of the file:
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@@
 <part name="JP9" library="SparkFun-Jumpers" deviceset="JUMPER-SMT_3_2-NC_TRACE" device="_SILK" package3d_urn="urn:adsk.eagle:package:39289/1" value="JUMPER-SMT_3_2-NC_TRACE_SILK"/>
 <part name="E2" library="SparkFun-RF" deviceset="ANTENNA-SMA-GROUNDED" device="EDGE_RPSMA" value="RP-SMA"/>
+<part name="S1" library="SparkFun-Switches" deviceset="MOMENTARY-SWITCH-SPST" device="-SMD-RIGHT-ANGLE" value="Reset"/>
+<part name="GND9" library="SparkFun-PowerSymbols" deviceset="GND" device=""/>
 </parts>
 <sheets>
@@
 <text x="182.88" y="175.26" size="1.524" layer="97" ratio="15">Microstrip Calculation:</text>
 <text x="63.5" y="63.5" size="2.54" layer="94" rot="MR180" align="center">USB</text>
-<text x="112.522" y="166.878" size="1.016" layer="97" align="top-left">PB22/23 are TXD/RXD to the EDBG</text>
-<text x="112.522" y="171.958" size="1.016" layer="97" align="top-left">PB10/11 are MOSI/SCK to SPI header.</text>
-<text x="112.268" y="218.44" size="1.016" layer="97" align="center-left">PA12 is SPI MISO (on SPI header).</text>
-<text x="112.268" y="215.9" size="1.016" layer="97" align="center-left">PA13 is DGI GPIO0 (goes to EDBG).</text>
-<text x="42.418" y="193.04" size="1.016" layer="97" align="center-right">PA5 is A4</text>
-<text x="42.418" y="185.42" size="1.016" layer="97" align="center-right">PB2 is A5</text>
 <text x="73.66" y="264.16" size="2.54" layer="94" font="vector" align="center">ATSAMD21G</text>
 <text x="254.254" y="63.246" size="2.54" layer="94" font="vector" align="center">Qwiic</text>
 <text x="332.74" y="200.66" size="2.54" layer="94" align="center">Cortex Debug/Program Connector</text>
 <text x="325.12" y="254" size="1.778" layer="97" align="center">I2C Pull Ups</text>
+<text x="81.28" y="289.56" size="1.27" layer="91">Do we need to move the TX/RX LEDs from the USB so they work during external radio connection?</text>
+<text x="81.28" y="284.48" size="1.27" layer="91">Add train button</text>
+<text x="81.28" y="287.02" size="1.27" layer="91">Add PTH holes for GPIO</text>
+<text x="118.11" y="182.88" size="0.762" layer="97" align="center">Bootloader TX LED</text>
+<text x="36.83" y="182.88" size="0.762" layer="97" align="center">Bootloader RX LED</text>
+<text x="81.28" y="281.94" size="1.27" layer="91">Add CTS RTS connections to GPIOs</text>
 </plain>
 <instances>
@@
 <instance part="FID4" gate="G$1" x="426.72" y="40.64" smashed="yes"/>
 <instance part="LOGO5" gate="G$1" x="337.82" y="45.72" smashed="yes"/>
-<instance part="GND32" gate="1" x="162.56" y="215.9" smashed="yes" rot="MR0">
-<attribute name="VALUE" x="162.56" y="215.646" size="1.778" layer="96" rot="MR0" align="top-center"/>
+<instance part="GND32" gate="1" x="162.56" y="218.44" smashed="yes" rot="MR0">
+<attribute name="VALUE" x="162.56" y="218.186" size="1.778" layer="96" rot="MR0" align="top-center"/>
 </instance>
 <instance part="GND50" gate="1" x="170.18" y="205.74" smashed="yes" rot="MR0">
@@
 <attribute name="VALUE" x="162.052" y="223.774" size="1.778" layer="96" font="vector" rot="MR0"/>
 </instance>
+<instance part="S1" gate="G$1" x="50.8" y="119.38" smashed="yes" rot="R90">
+<attribute name="NAME" x="49.276" y="119.38" size="1.778" layer="95" font="vector" rot="R90" align="bottom-center"/>
+<attribute name="VALUE" x="51.308" y="119.38" size="1.778" layer="96" font="vector" rot="R90" align="top-center"/>
+</instance>
+<instance part="GND9" gate="1" x="50.8" y="109.22" smashed="yes">
+<attribute name="VALUE" x="50.8" y="108.966" size="1.778" layer="96" align="top-center"/>
+</instance>
 </instances>
 <busses>
@@
 <segment>
 <pinref part="GND32" gate="1" pin="GND"/>
-<wire x1="162.56" y1="223.52" x2="162.56" y2="218.44" width="0.1524" layer="91"/>
+<wire x1="162.56" y1="223.52" x2="162.56" y2="220.98" width="0.1524" layer="91"/>
 <pinref part="E2" gate="G$1" pin="GND"/>
 </segment>
@@
 <pinref part="GND11" gate="1" pin="GND"/>
 </segment>
+<segment>
+<pinref part="S1" gate="G$1" pin="1"/>
+<pinref part="GND9" gate="1" pin="GND"/>
+<wire x1="50.8" y1="111.76" x2="50.8" y2="114.3" width="0.1524" layer="91"/>
+</segment>
 </net>
 <net name="3.3V" class="1">
@@
 </segment>
 </net>
-<net name="SPI_SCK" class="0">
+<net name="D13/SPI_SCK" class="0">
 <segment>
 <wire x1="218.44" y1="220.98" x2="220.98" y2="220.98" width="0.1524" layer="91"/>
@@
 </segment>
 </net>
-<net name="SPI_PICO" class="0">
+<net name="D11/SPI_PICO" class="0">
 <segment>
 <wire x1="218.44" y1="226.06" x2="220.98" y2="226.06" width="0.1524" layer="91"/>
@@
 </segment>
 </net>
-<net name="SPI_POCI" class="0">
+<net name="D12/SPI_POCI" class="0">
 <segment>
 <wire x1="218.44" y1="223.52" x2="220.98" y2="223.52" width="0.1524" layer="91"/>
@@
 </segment>
 </net>
-<net name="BOARD_ID" class="0">
+<net name="A2/BOARD_ID" class="0">
 <segment>
 <pinref part="R2" gate="G$1" pin="1"/>
@@
 </segment>
 </net>
-<net name="A3" class="0">
+<net name="A3/TRAIN" class="0">
 <segment>
 <pinref part="U2" gate="G$1" pin="PA04(AIN4/REFB/SER0:0/TC0:0)"/>
 <wire x1="43.18" y1="195.58" x2="40.64" y2="195.58" width="0.1524" layer="91"/>
 <label x="40.64" y="195.58" size="1.27" layer="95" rot="R180" xref="yes"/>
+</segment>
+<segment>
+<pinref part="S1" gate="G$1" pin="2"/>
+<wire x1="50.8" y1="124.46" x2="50.8" y2="127" width="0.1524" layer="91"/>
+<label x="50.8" y="127" size="1.27" layer="95" rot="R90" xref="yes"/>
 </segment>
 </net>
@@
 <net name="RX_LED" class="0">
 <segment>
-<pinref part="U2" gate="G$1" pin="PB03(AIN11/SER5:1)"/>
-<wire x1="43.18" y1="182.88" x2="40.64" y2="182.88" width="0.1524" layer="91"/>
-<label x="40.64" y="182.88" size="1.27" layer="95" rot="R180" xref="yes"/>
-</segment>
-<segment>
 <pinref part="D3" gate="G$1" pin="C"/>
 <wire x1="109.22" y1="106.68" x2="111.76" y2="106.68" width="0.1524" layer="91"/>
@@
 <net name="TX_LED" class="0">
 <segment>
-<pinref part="U2" gate="G$1" pin="PA27"/>
-<wire x1="111.76" y1="182.88" x2="114.3" y2="182.88" width="0.1524" layer="91"/>
-<label x="114.3" y="182.88" size="1.27" layer="95" xref="yes"/>
-</segment>
-<segment>
 <pinref part="D2" gate="G$1" pin="C"/>
 <wire x1="93.98" y1="109.22" x2="93.98" y2="106.68" width="0.1524" layer="91"/>
@@
 </segment>
 </net>
+<net name="A5" class="0">
+<segment>
+<pinref part="U2" gate="G$1" pin="PB02(AIN10/SER5:0)"/>
+<wire x1="43.18" y1="185.42" x2="40.64" y2="185.42" width="0.1524" layer="91"/>
+<label x="40.64" y="185.42" size="1.27" layer="95" rot="R180" xref="yes"/>
+</segment>
+</net>
+<net name="A4" class="0">
+<segment>
+<pinref part="U2" gate="G$1" pin="PA05(AIN5/SER0:1/TC0:1)"/>
+<wire x1="43.18" y1="193.04" x2="40.64" y2="193.04" width="0.1524" layer="91"/>
+<label x="40.64" y="193.04" size="1.27" layer="95" rot="R180" xref="yes"/>
+</segment>
+</net>
+<net name="D30" class="0">
+<segment>
+<pinref part="U2" gate="G$1" pin="PB22(SER5:2+)"/>
+<wire x1="111.76" y1="165.1" x2="114.3" y2="165.1" width="0.1524" layer="91"/>
+<label x="114.3" y="165.1" size="1.27" layer="95" xref="yes"/>
+</segment>
+</net>
+<net name="D31" class="0">
+<segment>
+<pinref part="U2" gate="G$1" pin="PB23(SER5:3+)"/>
+<wire x1="111.76" y1="162.56" x2="114.3" y2="162.56" width="0.1524" layer="91"/>
+<label x="114.3" y="162.56" size="1.27" layer="95" xref="yes"/>
+</segment>
+</net>

Commit message: Add train button, TX/RX LEDs, CTS/RTS connections, GPIO breakout. Increase to v11.
Parts:
- added J6: (no value), SparkFun-Connectors:CONN_021X02_NO_SILK
- D6: value PESD0402-0402T -> PESD0402
- S1: value Reset -> Train
Connections:
- net AREF renamed D42/AREF
- net SCL renamed D21/SCL
- net SDA renamed D20/SDA
- net USB_D+ renamed D29/USB_D+
- net USB_D- renamed D28/USB_D-
- net USB_HOST_EN renamed D27/USB_HOST_EN
- removed net A5: U2.PB02(AIN10/SER5:0)
- removed net CTS-I: J2.3
- removed net D30: U2.PB22(SER5:2+)
- removed net D31: U2.PB23(SER5:3+)
- removed net LORA_D2: U4.DIO2
- removed net N$5: D2.A, R5.1
- removed net N$9: D3.A, R12.1
- removed net RTS-O: J2.2
- removed net RX_LED: D3.C
- removed net TX_LED: D2.C
- new net A5/RX_LED: D3.A, U2.PB02(AIN10/SER5:0)
- new net D22: U2.PA12(I2C/SER2:0+)
- new net D23: U2.PB10(SER4:2+)
- new net D24: U2.PB11(SER4:3+)
- new net D30/CTS-I: J2.3, U2.PB22(SER5:2+)
- new net D31/TX_LED: D2.A, U2.PB23(SER5:3+)
- new net D38/RTS-O: J2.2, U2.PA13(I2C/SER2:1+)
- new net N$3: D3.C, R12.2
- new net N$4: D2.C, R5.2
- net 3.3V: no longer R12.2, R5.2
- net A0: now also J6.2
- net A1: now also J6.1
- net A3/TRAIN: now also S1.1; no longer S1.2
- net GND: now also R12.1, R5.1, S1.2; no longer S1.1
Other:
- note added: "Buttons, LEDs, ID"
- note added: "Cortex Debug"
- note added: "GPIO"
- note added: "I²C Pull Ups"
- note added: "Waveguide Calculation:"
- note removed: "Add CTS RTS connections to GPIOs"
- note removed: "Add PTH holes for GPIO"
- note removed: "Add train button"
- note removed: "Cortex Debug/Program Connector"
- note removed: "Do we need to move the TX/RX LEDs from the USB so they work during external radio connection?"
- note removed: "I2C Pull Ups"
- note removed: "Microstrip Calculation:"
- moved on the sheet: BYP, C12, C13, C14, C15, C16, C19, C3, C4, D2, D4, D5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

Commit message: Fix reversed pinout on locking JST.
Parts:
- removed J2: (no value), SparkFun-Connectors:CONN_06JST-SMD-LOCKING
- added J5: (no value), SparkFun-Connectors:CONN_06JST-SMD-LOCKING
Connections:
- net 5V: now also J5.1; no longer J2.6
- net D30/CTS-I: now also J5.4; no longer J2.3
- net D38/RTS-O: now also J5.5; no longer J2.2
- net GND: now also J5.6; no longer J2.1
- net RX-I: now also J5.2; no longer J2.5
- net TX-O: now also J5.3; no longer J2.4
Changed lines of the file:
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@@
 <part name="SUPPLY17" library="SparkFun-PowerSymbols" deviceset="V_USB" device=""/>
 <part name="SUPPLY4" library="SparkFun-PowerSymbols" deviceset="5V" device=""/>
-<part name="J2" library="SparkFun-Connectors" deviceset="CONN_06" device="JST-SMD-LOCKING"/>
 <part name="F1" library="SparkFun-Fuses" deviceset="PPTC" device="_6V500MA" value="6V 0.5A"/>
 <part name="D4" library="SparkFun-LED" deviceset="LED-BLUE" device="0603" value="BLUE"/>
@@
 <part name="GND13" library="SparkFun-PowerSymbols" deviceset="GND" device=""/>
 <part name="J6" library="SparkFun-Connectors" deviceset="CONN_02" device="1X02_NO_SILK"/>
+<part name="J5" library="SparkFun-Connectors" deviceset="CONN_06" device="JST-SMD-LOCKING"/>
 </parts>
 <sheets>
@@
 <attribute name="VALUE" x="231.14" y="48.514" size="1.778" layer="96" rot="MR0" align="bottom-center"/>
 </instance>
-<instance part="J2" gate="G$1" x="223.52" y="35.56" smashed="yes">
-<attribute name="VALUE" x="218.44" y="25.654" size="1.778" layer="96" font="vector"/>
-<attribute name="NAME" x="218.44" y="46.228" size="1.778" layer="95" font="vector"/>
-</instance>
 <instance part="F1" gate="F1" x="88.9" y="43.18" smashed="yes">
 <attribute name="NAME" x="90.17" y="48.768" size="1.778" layer="95" font="vector" align="bottom-center"/>
@@
 <attribute name="VALUE" x="269.24" y="30.734" size="1.778" layer="96" font="vector"/>
 <attribute name="NAME" x="269.24" y="41.148" size="1.778" layer="95" font="vector"/>
+</instance>
+<instance part="J5" gate="G$1" x="223.52" y="38.1" smashed="yes" rot="MR180">
+<attribute name="VALUE" x="218.44" y="48.006" size="1.778" layer="96" font="vector" rot="MR180"/>
+<attribute name="NAME" x="218.44" y="27.432" size="1.778" layer="95" font="vector" rot="MR180"/>
 </instance>
 </instances>
@@
 <wire x1="231.14" y1="30.48" x2="231.14" y2="27.94" width="0.1524" layer="91"/>
 <pinref part="GND4" gate="1" pin="GND"/>
-<pinref part="J2" gate="G$1" pin="1"/>
+<pinref part="J5" gate="G$1" pin="6"/>
 </segment>
 <segment>
@@
 <wire x1="231.14" y1="43.18" x2="231.14" y2="45.72" width="0.1524" layer="91"/>
 <pinref part="SUPPLY4" gate="G$1" pin="5V"/>
-<pinref part="J2" gate="G$1" pin="6"/>
+<pinref part="J5" gate="G$1" pin="1"/>
 </segment>
 </net>
@@
 <wire x1="228.6" y1="40.64" x2="231.14" y2="40.64" width="0.1524" layer="91"/>
 <label x="231.14" y="40.64" size="1.27" layer="95" rot="MR180" xref="yes"/>
-<pinref part="J2" gate="G$1" pin="5"/>
+<pinref part="J5" gate="G$1" pin="2"/>
 </segment>
 <segment>
@@
 <wire x1="228.6" y1="38.1" x2="231.14" y2="38.1" width="0.1524" layer="91"/>
 <label x="231.14" y="38.1" size="1.27" layer="95" rot="MR180" xref="yes"/>
-<pinref part="J2" gate="G$1" pin="4"/>
+<pinref part="J5" gate="G$1" pin="3"/>
 </segment>
 <segment>
@@
 </segment>
 <segment>
-<pinref part="J2" gate="G$1" pin="3"/>
 <label x="231.14" y="35.56" size="1.27" layer="95" xref="yes"/>
 <wire x1="228.6" y1="35.56" x2="231.14" y2="35.56" width="0.1524" layer="91"/>
+<pinref part="J5" gate="G$1" pin="4"/>
 </segment>
 </net>
@@
 </segment>
 <segment>
-<pinref part="J2" gate="G$1" pin="2"/>
 <wire x1="228.6" y1="33.02" x2="231.14" y2="33.02" width="0.1524" layer="91"/>
 <label x="231.14" y="33.02" size="1.27" layer="95" xref="yes"/>
-</segment>
-</net>
+<pinref part="J5" gate="G$1" pin="5"/>
+</segment>
+</net>

Commit message: Add display AES key. Always echo serial during AT config.
Other:
- note added: "Make Radio connector compatible with 5V signals"
Changed lines of the file:
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@@
 <wire x1="0" y1="76.2" x2="147.32" y2="76.2" width="0.2032" layer="97" style="longdash"/>
 <wire x1="360.68" y1="76.2" x2="360.68" y2="149.86" width="0.2032" layer="97" style="longdash"/>
+<text x="200.66" y="302.26" size="1.27" layer="91">Make Radio connector compatible with 5V signals</text>
 </plain>
 <instances>
