File: Hardware/868MHz/SparkFun LoRaSerial 868MHz - 1W.sch (EAGLE design)
At the start: 96 parts, among them J1 QWIIC_RIGHT_ANGLE, J3 USB C, J4 JTAG, Q1 20V/0.2A/8MHz/1.2Ω/1Vth, Q2 20V/0.2A/8MHz/1.2Ω/1Vth, Q3 600mA/40V, Q4 600mA/40V, Q5 600mA/40V, Q6 600mA/40V, Q8 20V/4.2A/52mΩ/1.4W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

Commit message: Change 868MHz connector to SMA
Parts:
- E2: device SparkFun-RF:ANTENNA-SMA-GROUNDEDEDGE_RPSMA -> SparkFun-RF:ANTENNA-SMA-GROUNDEDEDGE_SMA
Changed lines of the file:
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@@
 <part name="SUPPLY9" library="SparkFun-PowerSymbols" deviceset="3.3V" device=""/>
 <part name="JP9" library="SparkFun-Jumpers" deviceset="JUMPER-SMT_3_2-NC_TRACE" device="_SILK" package3d_urn="urn:adsk.eagle:package:39289/1" value="JUMPER-SMT_3_2-NC_TRACE_SILK"/>
-<part name="E2" library="SparkFun-RF" deviceset="ANTENNA-SMA-GROUNDED" device="EDGE_RPSMA" value="RP-SMA"/>
+<part name="E2" library="SparkFun-RF" deviceset="ANTENNA-SMA-GROUNDED" device="EDGE_SMA" value="RP-SMA"/>
 <part name="S1" library="SparkFun-Switches" deviceset="MOMENTARY-SWITCH-SPST" device="-SMD-RIGHT-ANGLE" value="Train"/>
 <part name="GND9" library="SparkFun-PowerSymbols" deviceset="GND" device=""/>

Commit message: Update schematics with flow control notes
Connections:
- net CTS-I_HV renamed !CTS!-I_HV
- net D30/CTS-I_LV renamed D30/!CTS!-I_LV
- net D38/RTS-O renamed D38/!RTS!-O
Other:
- note added: "Based on SAMD21 datasheet, section 25.6.3.2 Hardware Handshaking"
- note added: "If !CTS! is low, LoRaSerial will send data."
- note added: "LoRaSerial will drive !RTS! low when it is ready for data."
- note added: "When flow control is enabled:"
Changed lines of the file:
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@@
 <text x="5.08" y="129.54" size="1.778" layer="97" align="center-left">868MHz: 3.3/10</text>
 <text x="5.08" y="127" size="1.778" layer="97" align="center-left">433MHz: 10/20</text>
+<text x="226.06" y="7.62" size="1.27" layer="97" font="vector" align="center">LoRaSerial will drive !RTS! low when it is ready for data.</text>
+<text x="226.06" y="5.08" size="1.27" layer="97" font="vector" align="center">If !CTS! is low, LoRaSerial will send data.</text>
+<text x="226.06" y="2.54" size="1.27" layer="97" font="vector" align="center">Based on SAMD21 datasheet, section 25.6.3.2 Hardware Handshaking</text>
+<text x="226.06" y="10.16" size="1.27" layer="97" font="vector" align="center">When flow control is enabled:</text>
 </plain>
 <instances>
@@
 </segment>
 </net>
-<net name="D30/CTS-I_LV" class="0">
+<net name="D30/!CTS!-I_LV" class="0">
 <segment>
 <pinref part="U2" gate="G$1" pin="PB22(SER5:2+)"/>
@@
 </segment>
 </net>
-<net name="D38/RTS-O" class="0">
+<net name="D38/!RTS!-O" class="0">
 <segment>
 <pinref part="U2" gate="G$1" pin="PA13(I2C/SER2:1+)"/>
@@
 </segment>
 </net>
-<net name="CTS-I_HV" class="0">
+<net name="!CTS!-I_HV" class="0">
 <segment>
 <label x="175.26" y="20.32" size="1.27" layer="95" font="vector" xref="yes"/>
